File: res/kicad/bluepill_ethernet.sch (KiCad schematic (older format))
At the start: 47 parts, among them J1 HEADER-1x20, J2 Conn_01x03, J3 Conn_02x05_Odd_Even, J4 HEADER-1x20, J5 Conn_02x02_Odd_Even, J7 Conn_02x04_Odd_Even, SW1 SW_Push, U1 BluePill_STM32F103C, U2 93C46, U3 WIZ850io, U4 93C46, U5 PCF8574A, U6 LM75B

Commit message: Add values for caps, resistotrs, ... for board rev 3.1
Parts:
- C1, C3, C5, C7: value C -> 100nF
- C2, C4, C6: value CP -> 47µF
- R1, R2, R3, R4, R5, R6, R7, R8: value R -> 680Ω
- RN2: value 4,7k -> 4,7kΩ
Other:
- moved on the sheet: C3, R1, R2, R3, R5, R6, R7, R8
Changed lines of the file:
@@
 P 10150 5600
 F 0 "C4" H 10175 5700 50  0000 L CNN
-F 1 "CP" H 10175 5500 50  0000 L CNN
+F 1 "47µF" H 10175 5500 50  0000 L CNN
 F 2 "Capacitors_THT:CP_Radial_D4.0mm_P2.00mm" H 10188 5450 50  0001 C CNN
 F 3 "" H 10150 5600 50  0001 C CNN
@@
 P 9900 2750
 F 0 "C6" H 9782 2704 50  0000 R CNN
-F 1 "CP" H 9782 2795 50  0000 R CNN
+F 1 "47µF" H 9782 2795 50  0000 R CNN
 F 2 "Capacitors_THT:CP_Radial_D4.0mm_P2.00mm" H 9938 2600 50  0001 C CNN
 F 3 "" H 9900 2750 50  0001 C CNN
@@
 P 3650 900
 F 0 "C1" H 3675 1000 50  0000 L CNN
-F 1 "C" H 3675 800 50  0000 L CNN
+F 1 "100nF" H 3675 800 50  0000 L CNN
 F 2 "Capacitors_THT:C_Disc_D4.3mm_W1.9mm_P5.00mm" H 3688 750 50  0001 C CNN
 F 3 "" H 3650 900 50  0001 C CNN
@@
 P 5450 6600
 F 0 "C5" H 5475 6700 50  0000 L CNN
-F 1 "C" H 5475 6500 50  0000 L CNN
+F 1 "100nF" H 5475 6500 50  0000 L CNN
 F 2 "Capacitors_THT:C_Disc_D4.3mm_W1.9mm_P5.00mm" H 5488 6450 50  0001 C CNN
 F 3 "" H 5450 6600 50  0001 C CNN
@@
 P 11050 900
 F 0 "C2" H 11075 1000 50  0000 L CNN
-F 1 "CP" H 11075 800 50  0000 L CNN
+F 1 "47µF" H 11075 800 50  0000 L CNN
 F 2 "Capacitors_THT:CP_Radial_D4.0mm_P2.00mm" H 11088 750 50  0001 C CNN
 F 3 "" H 11050 900 50  0001 C CNN
@@
 P 9900 2450
 F 0 "C7" H 9925 2550 50  0000 L CNN
-F 1 "C" H 9925 2350 50  0000 L CNN
+F 1 "100nF" H 9925 2350 50  0000 L CNN
 F 2 "Capacitors_THT:C_Disc_D4.3mm_W1.9mm_P5.00mm" H 9938 2300 50  0001 C CNN
 F 3 "" H 9900 2450 50  0001 C CNN
@@
 P 10450 850
 F 0 "RN2" H 9970 896 50  0000 R CNN
-F 1 "4,7k" H 9970 805 50  0000 R CNN
+F 1 "4,7kΩ" H 9970 805 50  0000 R CNN
 F 2 "Resistor_THT:R_Array_SIP9" V 10925 850 50  0001 C CNN
 F 3 "http://www.vishay.com/docs/31509/csc.pdf" H 10450 850 50  0001 C CNN
@@
 $EndComp
 Wire Wire Line
-	2250 4550 2500 5150
+	2250 4550 2500 4550
 $Comp
 L Device:LED D4
@@
 $EndComp
 Wire Wire Line
-	2500 5250 2250 4850
-Wire Wire Line
-	2250 5150 2500 5350
+	2500 4850 2250 4850
+Wire Wire Line
+	2250 5150 2500 5150
 Wire Wire Line
 	2500 5450 2250 5450
 Wire Wire Line
-	2250 5750 2500 5550
-Wire Wire Line
-	2500 5650 2250 6050
-Wire Wire Line
-	2250 6350 2500 5750
-Wire Wire Line
-	2500 5850 2250 6650
+	2250 5750 2500 5750
+Wire Wire Line
+	2500 6050 2250 6050
+Wire Wire Line
+	2250 6350 2500 6350
+Wire Wire Line
+	2500 6650 2250 6650
 Wire Wire Line
 	600  3900 600  5150
@@
 	1300 4500 2900 4500
 Wire Wire Line
-	2900 4500 2900 5150
+	2900 4500 2900 4550
 Connection ~ 1300 4500
 Wire Wire Line
@@
 L Device:R R1
 U 1 1 5F8367EB
+P 2650 4550
+F 0 "R1" V 2443 4550 50  0000 C CNN
+F 1 "680Ω" V 2534 4550 50  0000 C CNN
+F 2 "Resistor_SMD:R_0805_2012Metric" V 2580 4550 50  0001 C CNN
+F 3 "~" H 2650 4550 50  0001 C CNN
+	1    2650 4550
+	0    1    1    0
+$EndComp
+$Comp
+L Device:R R2
+U 1 1 5F83AB09
+P 2650 4850
+F 0 "R2" V 2443 4850 50  0000 C CNN
+F 1 "680Ω" V 2534 4850 50  0000 C CNN
+F 2 "Resistor_SMD:R_0805_2012Metric" V 2580 4850 50  0001 C CNN
+F 3 "~" H 2650 4850 50  0001 C CNN
+	1    2650 4850
+	0    1    1    0
+$EndComp
+$Comp
+L Device:R R3
+U 1 1 5F83AD2B
 P 2650 5150
-F 0 "R1" V 2443 5150 50  0000 C CNN
-F 1 "R" V 2534 5150 50  0000 C CNN
+F 0 "R3" V 2443 5150 50  0000 C CNN
+F 1 "680Ω" V 2534 5150 50  0000 C CNN
 F 2 "Resistor_SMD:R_0805_2012Metric" V 2580 5150 50  0001 C CNN
 F 3 "~" H 2650 5150 50  0001 C CNN
 	1    2650 5150
-	0    1    1    0
-$EndComp
-$Comp
-L Device:R R2
-U 1 1 5F83AB09
-P 2650 5250
-F 0 "R2" V 2443 5250 50  0000 C CNN
-F 1 "R" V 2534 5250 50  0000 C CNN
-F 2 "Resistor_SMD:R_0805_2012Metric" V 2580 5250 50  0001 C CNN
-F 3 "~" H 2650 5250 50  0001 C CNN
-	1    2650 5250
-	0    1    1    0
-$EndComp
-$Comp
-L Device:R R3
-U 1 1 5F83AD2B
-P 2650 5350
-F 0 "R3" V 2443 5350 50  0000 C CNN
-F 1 "R" V 2534 5350 50  0000 C CNN
-F 2 "Resistor_SMD:R_0805_2012Metric" V 2580 5350 50  0001 C CNN
-F 3 "~" H 2650 5350 50  0001 C CNN
-	1    2650 5350
 	0    1    1    0
 $EndComp
@@
 P 2650 5450
 F 0 "R4" V 2443 5450 50  0000 C CNN
-F 1 "R" V 2534 5450 50  0000 C CNN
+F 1 "680Ω" V 2534 5450 50  0000 C CNN
 F 2 "Resistor_SMD:R_0805_2012Metric" V 2580 5450 50  0001 C CNN
 F 3 "~" H 2650 5450 50  0001 C CNN
@@
 L Device:R R5
 U 1 1 5F83B1A6
-P 2650 5550
-F 0 "R5" V 2443 5550 50  0000 C CNN
-F 1 "R" V 2534 5550 50  0000 C CNN
-F 2 "Resistor_SMD:R_0805_2012Metric" V 2580 5550 50  0001 C CNN
-F 3 "~" H 2650 5550 50  0001 C CNN
-	1    2650 5550
-	0    1    1    0
-$EndComp
-$Comp
-L Device:R R6
-U 1 1 5F83B3B4
-P 2650 5650
-F 0 "R6" V 2443 5650 50  0000 C CNN
-F 1 "R" V 2534 5650 50  0000 C CNN
-F 2 "Resistor_SMD:R_0805_2012Metric" V 2580 5650 50  0001 C CNN
-F 3 "~" H 2650 5650 50  0001 C CNN
-	1    2650 5650
-	0    1    1    0
-$EndComp
-$Comp
-L Device:R R7
-U 1 1 5F83B558
 P 2650 5750
-F 0 "R7" V 2443 5750 50  0000 C CNN
-F 1 "R" V 2534 5750 50  0000 C CNN
+F 0 "R5" V 2443 5750 50  0000 C CNN
+F 1 "680Ω" V 2534 5750 50  0000 C CNN
 F 2 "Resistor_SMD:R_0805_2012Metric" V 2580 5750 50  0001 C CNN
 F 3 "~" H 2650 5750 50  0001 C CNN
@@
 $EndComp
 $Comp
+L Device:R R6
+U 1 1 5F83B3B4
+P 2650 6050
+F 0 "R6" V 2443 6050 50  0000 C CNN
+F 1 "680Ω" V 2534 6050 50  0000 C CNN
+F 2 "Resistor_SMD:R_0805_2012Metric" V 2580 6050 50  0001 C CNN
+F 3 "~" H 2650 6050 50  0001 C CNN
+	1    2650 6050
+	0    1    1    0
+$EndComp
+$Comp
+L Device:R R7
+U 1 1 5F83B558
+P 2650 6350
+F 0 "R7" V 2443 6350 50  0000 C CNN
+F 1 "680Ω" V 2534 6350 50  0000 C CNN
+F 2 "Resistor_SMD:R_0805_2012Metric" V 2580 6350 50  0001 C CNN
+F 3 "~" H 2650 6350 50  0001 C CNN
+	1    2650 6350
+	0    1    1    0
+$EndComp
+$Comp
 L Device:R R8
 U 1 1 5F83B73C
-P 2650 5850
-F 0 "R8" V 2443 5850 50  0000 C CNN
-F 1 "R" V 2534 5850 50  0000 C CNN
-F 2 "Resistor_SMD:R_0805_2012Metric" V 2580 5850 50  0001 C CNN
-F 3 "~" H 2650 5850 50  0001 C CNN
-	1    2650 5850
-	0    1    1    0
-$EndComp
-Wire Wire Line
-	2800 5850 2900 5850
+P 2650 6650
+F 0 "R8" V 2443 6650 50  0000 C CNN
+F 1 "680Ω" V 2534 6650 50  0000 C CNN
+F 2 "Resistor_SMD:R_0805_2012Metric" V 2580 6650 50  0001 C CNN
+F 3 "~" H 2650 6650 50  0001 C CNN
+	1    2650 6650
+	0    1    1    0
+$EndComp
+Wire Wire Line
+	2800 6650 2900 6650
+Wire Wire Line
+	2800 6350 2900 6350
+Connection ~ 2900 6350
+Wire Wire Line
+	2900 6350 2900 6650
+Wire Wire Line
+	2900 6050 2800 6050
+Connection ~ 2900 6050
+Wire Wire Line
+	2900 6050 2900 6350
 Wire Wire Line
 	2800 5750 2900 5750
 Connection ~ 2900 5750
 Wire Wire Line
-	2900 5750 2900 5850
-Wire Wire Line
-	2900 5650 2800 5650
-Connection ~ 2900 5650
-Wire Wire Line
-	2900 5650 2900 5750
-Wire Wire Line
-	2800 5550 2900 5550
-Connection ~ 2900 5550
-Wire Wire Line
-	2900 5550 2900 5650
+	2900 5750 2900 6050
 Wire Wire Line
 	2900 5450 2800 5450
 Connection ~ 2900 5450
 Wire Wire Line
-	2900 5450 2900 5550
-Wire Wire Line
-	2800 5350 2900 5350
-Connection ~ 2900 5350
-Wire Wire Line
-	2900 5350 2900 5450
-Wire Wire Line
-	2900 5250 2800 5250
-Connection ~ 2900 5250
-Wire Wire Line
-	2900 5250 2900 5350
+	2900 5450 2900 5750
 Wire Wire Line
 	2800 5150 2900 5150
 Connection ~ 2900 5150
 Wire Wire Line
-	2900 5150 2900 5250
+	2900 5150 2900 5450
+Wire Wire Line
+	2900 4850 2800 4850
+Connection ~ 2900 4850
+Wire Wire Line
+	2900 4850 2900 5150
+Wire Wire Line
+	2800 4550 2900 4550
+Connection ~ 2900 4550
+Wire Wire Line
+	2900 4550 2900 4850
 $Comp
 L Connector_Generic:Conn_02x04_Odd_Even J7
@@
 L bluepill_ethernet-rescue:C-device C3
 U 1 1 5FBB6638
-P 2900 6400
-F 0 "C3" H 2925 6500 50  0000 L CNN
-F 1 "C" H 2925 6300 50  0000 L CNN
-F 2 "Capacitor_SMD:C_0805_2012Metric" H 2938 6250 50  0001 C CNN
-F 3 "" H 2900 6400 50  0001 C CNN
-	1    2900 6400
-	1    0    0    -1
-$EndComp
-Wire Wire Line
-	2900 6250 2900 5850
-Connection ~ 2900 5850
-Wire Wire Line
-	2900 6550 2900 7000
+P 2900 6800
+F 0 "C3" H 2925 6900 50  0000 L CNN
+F 1 "100nF" H 2925 6700 50  0000 L CNN
+F 2 "Capacitor_SMD:C_0805_2012Metric" H 2938 6650 50  0001 C CNN
+F 3 "" H 2900 6800 50  0001 C CNN
+	1    2900 6800
+	1    0    0    -1
+$EndComp
+Connection ~ 2900 6650
+Wire Wire Line
+	2900 6950 2900 7000
 Connection ~ 2900 7000
 Wire Wire Line
